File: Joycon breakout pcb/Joycon breakout pcb.kicad_pcb (KiCad board)
At the start: 2 copper layers, 6 x 6 mm, 2 parts, among them J1 Conn_01x06_Female, J2 Conn_01x06_Male

Commit message: fixed Silkscreen
Other:
- board text added: "VCC"
- board text removed: "3.3V"
Changed lines of the file:
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@@
     (effects (font (size 0.6 0.6) (thickness 0.1)) (justify mirror))
   )
-  (gr_text "X Axis" (at 63.15 37.9) (layer B.SilkS)
+  (gr_text VCC (at 63.65 37.9) (layer B.SilkS)
     (effects (font (size 0.6 0.6) (thickness 0.1)) (justify mirror))
   )
-  (gr_text "Y Axis" (at 63.15 34.9) (layer B.SilkS)
+  (gr_text GND (at 63.65 34.9) (layer B.SilkS)
     (effects (font (size 0.6 0.6) (thickness 0.1)) (justify mirror))
   )
-  (gr_text GND (at 63.675 36.9) (layer B.SilkS)
+  (gr_text "Y Axis" (at 63.175 36.9) (layer B.SilkS)
     (effects (font (size 0.6 0.6) (thickness 0.1)) (justify mirror))
   )
-  (gr_text 3.3V (at 63.575 33.9) (layer B.SilkS)
+  (gr_text "X Axis" (at 63.15 33.9) (layer B.SilkS)
     (effects (font (size 0.6 0.6) (thickness 0.1)) (justify mirror))
   )
